File: KiCad 9 ESP32 demo project/esp32-c3-02.kicad_sch (KiCad schematic)
At the start: 0 parts

Commit message: schematic esp32 sheet
Parts:
- added C10: 0.1U, symbol Device:C
- added C11: 1U, symbol Device:C
- added C9: 4.7U, symbol Device:C_Polarized
- added J3: GSD090012SEU, GSD090012SEU:AMPHENOL_GSD090012SEU, symbol GSD090012SEU:GSD090012SEU
- added LED6: Green_LED, LTST-C170KRKT:DIOC200X125X110, symbol LTST-C170KRKT:LTST-C170KRKT
- added LED7: Red_LED, LTST-C170KRKT:DIOC200X125X110, symbol LTST-C170KRKT:LTST-C170KRKT
- added R11: 1K, symbol Device:R
- added R12: 22K1, symbol Device:R
- added R13: 47K5, symbol Device:R
- added R15, R20: 50R, symbol Device:R
- added R16, R18: 470R, symbol Device:R
- added U3: ESP32-C3-WROOM-02-H4, ESP32-C3-WROOM-02-H4:MODULE_ESP32-C3-WROOM-02-H4, symbol ESP32-C3-WROOM-02-H4:ESP32-C3-WROOM-02-H4
- added U4: CP2102N-Axx-xQFN20, Package_DFN_QFN:SiliconLabs_QFN-20-1EP_3x3mm_P0.5mm, symbol Interface_USB:CP2102N-Axx-xQFN20
- added U5: USBLC6-2SC6, Package_TO_SOT_SMD:SOT-23-6, symbol Power_Protection:USBLC6-2SC6
- added U6: W25Q32JVSSIQ, W25Q32JVSSIQ:SOIC127P790X216-8N, symbol W25Q32JVSSIQ:W25Q32JVSSIQ
Connections:
- new net: C11.1, R12.2, R13.1, U4.8 (VBUS)
- new net: R11.2, U4.9 (~{RST})
- new net: R16.1, U4.20 (~{TXT}/GPIO.2)
- new net: LED6.-, R16.2
- new net: R15.1, U3.6 (IO7)
- new net: R18.1, U4.19 (~{RXT}/GPIO.3)
- new net: LED7.-, R18.2
- new net: R20.2, U3.5 (IO6)
- new net +3.3V: C10.2, C9.1, LED6.+, LED7.+, R11.1, U4.6 (VDD), U4.7 (VREGIN)
- new net BOOT: U3.8 (IO9)
- new net CD_SD: U3.18 (IO0)
- new net CS: U3.10 (IO10)
- new net DTS: U4.15 (~{CTS})
- new net EN: U3.2 (EN)
- new net GND: C10.1, C11.2, C9.2, R13.2, U3.19 (GND), U3.20 (GND), U3.21 (GND), U3.22 (GND), U3.23 (GND), U3.24 (GND), U3.25 (GND), U3.26 (GND), U3.27 (GND), U3.28 (GND), U3.29 (GND), U3.30 (GND), U3.31 (GND), U3.32 (GND), U3.33 (GND), U3.34 (GND), U3.35 (GND), U3.36 (GND), U3.37 (GND), U3.38 (GND), U3.39 (GND), U3.9 (GND), U4.12 (GND), U4.21 (GND), U4.3 (GND), U5.2 (GND)
- new net GPIO18: U3.13 (IO18)
- new net GPIO8: U3.7 (IO8)
- new net GPOI19: U3.14 (IO19)
- new net MIC_OUT: U3.4 (IO5)
- new net MISO_DO: U3.16 (IO2)
- new net MOSI_DI: R15.2
- new net PHOTO_C: U3.17 (IO1)
- new net RTS: U4.16 (~{RTS})
- new net RX_TX: U3.12 (TXD), U4.17 (RXD)
- new net SCL: U3.15 (IO3)
- new net SCLK: R20.1
- new net SDA: U3.3 (IO4)
- new net TX_RX: U3.11 (RXD), U4.18 (TXD)
- new net USB_D+: U4.4 (D+), U5.3 (I/O2)
- new net USB_D-: U4.5 (D-), U5.1 (I/O1)
- new net USB_DN: U5.6 (I/O1)
- new net USB_DP: U5.4 (I/O2)
- new net VBUS: R12.1, U5.5 (VBUS)
- no-connect marks 0 -> 5
Other:
- note added: "USB Module"

Commit message: schematic esp32 done
Parts:
- added C12, C7: 10u, symbol Device:C_Polarized
- added C13, C14, C8: 0.1u, symbol Device:C
- added R16, R22: 50R, symbol Device:R
- added R19: 10K, symbol Device:R
- added TP1: Test MOSI, symbol Connector:TestPoint
- added TP2: Test MISO, symbol Connector:TestPoint
- added TP3: Test SCLK, symbol Connector:TestPoint
- added TP4: Test CS_SD, symbol Connector:TestPoint
- added TP5: Test CS, symbol Connector:TestPoint
Connections:
- net CD_SD is gone; now on net CS_SD: U3.18 (IO0)
- net +3.3V: now also U3.1 (3V3), U6.3 (~{WP}(IO2)), U6.7 (~{HOLD}/~{RESET}(IO3)), U6.8 (VCC), C14.1, C7.1, C8.1, R19.2
- net CS: now also U6.1 (~{CS}), TP5.1
- net GND: now also J3.3 (VSS1), J3.6 (VSS2), J3.8 (DAT1), J3.9 (DAT2), J3.G1 (SHIELD_GND), J3.G2 (SHIELD_GND__1), J3.G3 (SHIELD_GND__2), J3.G4 (SHIELD_GND__3), U6.4 (GND), C12.2, C13.2, C14.2, C7.2, C8.2
- net MISO_DO: now also R16.2, R22.1, TP2.1
- net MOSI_DI: now also J3.2 (CMD), U6.5 (DI(IO0)), TP1.1
- net SCLK: now also J3.5 (CLK), U6.6 (CLK), TP3.1
- net at U6.2 (DO(IO1)): now also R22.2
- net CS_SD: now reaches J3.1 (CD/DAT3)
- net CS_SD: now also R19.1, TP4.1
- net at J3.4 (VDD1): now also C12.1, C13.1
- net at J3.7 (DAT0): now also R16.1
- no-connect marks 5 -> 7
Other:
- added sheet Sensors (sensors.kicad_sch)
- added sheet User Interface (User_Interface.kicad_sch)
- note added: "ESP32-C3-WROOM-02-H4"
- note added: "Flash Memory"
- note added: "SD_Card_Module"
- note added: "Test Points"
- title: (none) -> ESP32-C3, USB and Flash Memory
- moved on the sheet: J3, R15, R20, U3, U6
