File: KiCad 9 ESP32 demo project/esp32-c3-02.kicad_sch (KiCad schematic)
At the start: 30 parts, among them J3 GSD090012SEU, U3 ESP32-C3-WROOM-02-H4, U4 CP2102N-Axx-xQFN20, U5 USBLC6-2SC6, U6 W25Q32JVSSIQ

Commit message: Schematic Done
Parts:
- C10, C11, C8: footprint (none) -> Capacitor_SMD:C_0805_2012Metric
- C12, C13, C14, R11, R12, R13, R15, R16, R18, R19, R20, R22: footprint (none) -> Resistor_SMD:R_0805_2012Metric
- C7, C9: footprint (none) -> T491A104K035AT:CAPC3216X110N
- J3: footprint GSD090012SEU:AMPHENOL_GSD090012SEU -> Connector_PinHeader_2.54mm:PinHeader_1x04_P2.54mm_Vertical
- LED6, LED7: footprint LTST-C170KRKT:DIOC200X125X110 -> Resistor_SMD:R_0805_2012Metric
- R14: renamed from R16; footprint (none) -> Resistor_SMD:R_0805_2012Metric
- TP1, TP2, TP3, TP4, TP5: footprint (none) -> TestPoint:TestPoint_Pad_D1.0mm
Connections:
- net DTS renamed DTR
Other:
- sheet Sensors ports: added MIC_OUT, PHOTO_C, SCL, SDA; removed none
- sheet User Interface ports: added BOOT, DTR, EN, GPIO18, GPIO19, GPIO8, RTS, SCL, SDA; removed none

Commit message: stated layout
Parts:
- C12, C13, C14: footprint Resistor_SMD:R_0805_2012Metric -> Capacitor_SMD:C_0805_2012Metric
- J3: footprint Connector_PinHeader_2.54mm:PinHeader_1x04_P2.54mm_Vertical -> GSD090012SEU:AMPHENOL_GSD090012SEU
- LED6, LED7: footprint Resistor_SMD:R_0805_2012Metric -> LTST-C170KRKT:DIOC200X125X110
- U4: footprint Package_DFN_QFN:SiliconLabs_QFN-20-1EP_3x3mm_P0.5mm -> Package_DFN_QFN:SiliconLabs_QFN-20-1EP_3x3mm_P0.5mm_EP1.8x1.8mm
Connections:
- net +3.3V: now also C12.1, C13.1, J3.4 (VDD1)
Other:
- moved on the sheet: TP1, TP2, TP3, TP4, TP5
Changed lines of the file:
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@@
 	)
 	(junction
+		(at 266.7 101.6)
+		(diameter 0)
+		(color 0 0 0 0)
+	)
+	(junction
 		(at 266.7 113.03)
 		(diameter 0)
@@
 	(wire
 		(pts
+			(xy 266.7 99.06) (xy 266.7 101.6)
+		)
+		(stroke
+			(width 0)
+			(type default)
+		)
+	)
+	(wire
+		(pts
 			(xy 22.86 160.02) (xy 53.34 160.02)
 		)
@@
 	)
 	(rectangle
-		(start 154.94 35.56)
-		(end 177.8 90.17)
+		(start 154.94 31.75)
+		(end 177.8 86.36)
 		(stroke
 			(width 0)
@@
 	(text "Test Points\n"
 		(exclude_from_sim no)
-		(at 160.02 33.274 0)
+		(at 160.02 29.464 0)
 		(effects
 			(font
@@
 	)
 	(label "MISO_DO"
-		(at 166.37 53.34 0)
+		(at 166.37 49.53 0)
 		(effects
 			(font
@@
 	)
 	(label "SCLK"
-		(at 166.37 63.5 0)
+		(at 166.37 59.69 0)
 		(effects
 			(font
@@
 	)
 	(label "CS"
-		(at 166.37 83.82 0)
+		(at 166.37 80.01 0)
 		(effects
 			(font
@@
 	)
 	(label "CS_SD"
-		(at 166.37 73.66 0)
+		(at 166.37 69.85 0)
 		(effects
 			(font
@@
 	)
 	(label "MOSI_DI"
-		(at 166.37 43.18 0)
+		(at 166.37 39.37 0)
 		(effects
 			(font
@@
 			)
 		)
-		(property "Footprint" "Resistor_SMD:R_0805_2012Metric"
+		(property "Footprint" "Capacitor_SMD:C_0805_2012Metric"
 			(at 96.2152 163.83 0)
 			(effects
@@
 	)
 	(symbol
+		(lib_id "power:+3.3V")
+		(at 266.7 99.06 0)
+		(unit 1)
+		(exclude_from_sim no)
+		(in_bom yes)
+		(on_board yes)
+		(dnp no)
+		(fields_autoplaced yes)
+		(property "Reference" "#PWR56"
+			(at 266.7 102.87 0)
+			(effects
+				(font
+					(size 1.27 1.27)
+				)
+				(hide yes)
+			)
+		)
+		(property "Value" "+3.3V"
+			(at 266.7 93.98 0)
+			(effects
+				(font
+					(size 1.27 1.27)
+				)
+			)
+		)
+		(property "Footprint" ""
+			(at 266.7 99.06 0)
+			(effects
+				(font
+					(size 1.27 1.27)
+				)
+				(hide yes)
+			)
+		)
+		(property "Datasheet" ""
+			(at 266.7 99.06 0)
+			(effects
+				(font
+					(size 1.27 1.27)
+				)
+				(hide yes)
+			)
+		)
+		(property "Description" "Power symbol creates a global label with name \"+3.3V\""
+			(at 266.7 99.06 0)
+			(effects
+				(font
+					(size 1.27 1.27)
+				)
+				(hide yes)
+			)
+		)
+		(pin "1"
+		)
+		(instances
+			(project "KiCad 9 ESP32 demo project"
+				(path "/80604368-af49-40dd-987f-c761cdff6830/4a22eb7a-047d-4a09-a619-875484efe01d"
+					(reference "#PWR56")
+					(unit 1)
+				)
+			)
+		)
+	)
+	(symbol
 		(lib_id "Device:R")
 		(at 55.88 67.31 90)
@@
 			)
 		)
-		(property "Footprint" "Resistor_SMD:R_0805_2012Metric"
+		(property "Footprint" "Capacitor_SMD:C_0805_2012Metric"
 			(at 262.5852 124.46 0)
 			(effects
@@
 	(symbol
 		(lib_id "Connector:TestPoint")
-		(at 166.37 63.5 90)
+		(at 166.37 59.69 90)
 		(unit 1)
 		(exclude_from_sim no)
@@
 		(fields_autoplaced yes)
 		(property "Reference" "TP3"
-			(at 163.068 58.42 90)
+			(at 163.068 54.61 90)
 			(effects
 				(font
@@
 		)
 		(property "Value" "Test SCLK"
-			(at 163.068 60.96 90)
+			(at 163.068 57.15 90)
 			(effects
 				(font
@@
 		)
 		(property "Footprint" "TestPoint:TestPoint_Pad_D1.0mm"
-			(at 166.37 58.42 0)
+			(at 166.37 54.61 0)
 			(effects
 				(font
@@
 		)
 		(property "Datasheet" "~"
-			(at 166.37 58.42 0)
+			(at 166.37 54.61 0)
 			(effects
 				(font
@@
 		)
 		(property "Description" "test point"
-			(at 166.37 63.5 0)
+			(at 166.37 59.69 0)
 			(effects
 				(font
@@
 			)
 		)
-		(property "Footprint" "Resistor_SMD:R_0805_2012Metric"
+		(property "Footprint" "LTST-C170KRKT:DIOC200X125X110"
 			(at 121.92 95.25 0)
 			(effects
@@
 			)
 		)
-		(property "Footprint" "Resistor_SMD:R_0805_2012Metric"
+		(property "Footprint" "Capacitor_SMD:C_0805_2012Metric"
 			(at 272.7452 124.46 0)
 			(effects
@@
 	(symbol
 		(lib_id "Connector:TestPoint")
-		(at 166.37 73.66 90)
+		(at 166.37 69.85 90)
 		(unit 1)
 		(exclude_from_sim no)
@@
 		(fields_autoplaced yes)
 		(property "Reference" "TP4"
-			(at 163.068 68.58 90)
+			(at 163.068 64.77 90)
 			(effects
 				(font
@@
 		)
 		(property "Value" "Test CS_SD"
-			(at 163.068 71.12 90)
+			(at 163.068 67.31 90)
 			(effects
 				(font
@@
 		)
 		(property "Footprint" "TestPoint:TestPoint_Pad_D1.0mm"
-			(at 166.37 68.58 0)
+			(at 166.37 64.77 0)
 			(effects
 				(font
@@
 		)
 		(property "Datasheet" "~"
-			(at 166.37 68.58 0)
+			(at 166.37 64.77 0)
 			(effects
 				(font
@@
 		)
 		(property "Description" "test point"
-			(at 166.37 73.66 0)
+			(at 166.37 69.85 0)
 			(effects
 				(font
@@
 		(dnp no)
 		(property "Reference" "R22"
-			(at 36.83 162.814 90)
+			(at 37.338 162.814 90)
 			(effects
 				(font
@@
 		)
 		(property "Value" "50R"
-			(at 42.418 162.814 90)
+			(at 43.942 162.814 90)
 			(effects
 				(font
@@
 	(symbol
 		(lib_id "Connector:TestPoint")
-		(at 166.37 83.82 90)
+		(at 166.37 80.01 90)
 		(unit 1)
 		(exclude_from_sim no)
@@
 		(fields_autoplaced yes)
 		(property "Reference" "TP5"
-			(at 163.068 78.74 90)
+			(at 163.068 74.93 90)
 			(effects
 				(font
@@
 		)
 		(property "Value" "Test CS"
-			(at 163.068 81.28 90)
+			(at 163.068 77.47 90)
 			(effects
 				(font
@@
 		)
 		(property "Footprint" "TestPoint:TestPoint_Pad_D1.0mm"
-			(at 166.37 78.74 0)
+			(at 166.37 74.93 0)
 			(effects
 				(font
@@
 		)
 		(property "Datasheet" "~"
-			(at 166.37 78.74 0)
+			(at 166.37 74.93 0)
 			(effects
 				(font
@@
 		)
 		(property "Description" "test point"
-			(at 166.37 83.82 0)
+			(at 166.37 80.01 0)
 			(effects
 				(font
@@
 			)
 		)
-		(property "Footprint" "Connector_PinHeader_2.54mm:PinHeader_1x04_P2.54mm_Vertical"
+		(property "Footprint" "GSD090012SEU:AMPHENOL_GSD090012SEU"
 			(at 214.63 114.3 0)
 			(effects
@@
 			)
 		)
-		(property "Footprint" "Resistor_SMD:R_0805_2012Metric"
+		(property "Footprint" "LTST-C170KRKT:DIOC200X125X110"
 			(at 121.92 109.22 0)
 			(effects
@@
 	(symbol
 		(lib_id "Connector:TestPoint")
-		(at 166.37 43.18 90)
+		(at 166.37 39.37 90)
 		(unit 1)
 		(exclude_from_sim no)
@@
 		(fields_autoplaced yes)
 		(property "Reference" "TP1"
-			(at 163.068 38.1 90)
+			(at 163.068 34.29 90)
 			(effects
 				(font
@@
 		)
 		(property "Value" "Test MOSI"
-			(at 163.068 40.64 90)
+			(at 163.068 36.83 90)
 			(effects
 				(font
@@
 		)
 		(property "Footprint" "TestPoint:TestPoint_Pad_D1.0mm"
-			(at 166.37 38.1 0)
+			(at 166.37 34.29 0)
 			(effects
 				(font
@@
 		)
 		(property "Datasheet" "~"
-			(at 166.37 38.1 0)
+			(at 166.37 34.29 0)
 			(effects
 				(font
@@
 		)
 		(property "Description" "test point"
-			(at 166.37 43.18 0)
+			(at 166.37 39.37 0)
 			(effects
 				(font
@@
 	(symbol
 		(lib_id "Connector:TestPoint")
-		(at 166.37 53.34 90)
+		(at 166.37 49.53 90)
 		(unit 1)
 		(exclude_from_sim no)
@@
 		(fields_autoplaced yes)
 		(property "Reference" "TP2"
-			(at 163.068 48.26 90)
+			(at 163.068 44.45 90)
 			(effects
 				(font
@@
 		)
 		(property "Value" "Test MISO"
-			(at 163.068 50.8 90)
+			(at 163.068 46.99 90)
 			(effects
 				(font
@@
 		)
 		(property "Footprint" "TestPoint:TestPoint_Pad_D1.0mm"
-			(at 166.37 48.26 0)
+			(at 166.37 44.45 0)
 			(effects
 				(font
@@
 		)
 		(property "Datasheet" "~"
-			(at 166.37 48.26 0)
+			(at 166.37 44.45 0)
 			(effects
 				(font
@@
 		)
 		(property "Description" "test point"
-			(at 166.37 53.34 0)
+			(at 166.37 49.53 0)
 			(effects
 				(font
@@
 			)
 		)
-		(property "Footprint" "Package_DFN_QFN:SiliconLabs_QFN-20-1EP_3x3mm_P0.5mm"
+		(property "Footprint" "Package_DFN_QFN:SiliconLabs_QFN-20-1EP_3x3mm_P0.5mm_EP1.8x1.8mm"
 			(at 109.22 116.84 0)
 			(effects

Commit message: power layout done
Changed lines of the file:
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@@
 		(lib_id "Device:C")
 		(at 39.37 87.63 0)
+		(mirror y)
 		(unit 1)
 		(exclude_from_sim no)
@@
 		(on_board yes)
 		(dnp no)
-		(fields_autoplaced yes)
 		(property "Reference" "C11"
-			(at 43.18 86.3599 0)
+			(at 35.56 86.3599 0)
 			(effects
 				(font
@@
 		)
 		(property "Value" "1U"
-			(at 43.18 88.8999 0)
+			(at 35.56 88.8999 0)
 			(effects
 				(font
@@
 		)
 		(property "Footprint" "Capacitor_SMD:C_0805_2012Metric"
-			(at 40.3352 91.44 0)
+			(at 38.4048 91.44 0)
 			(effects
 				(font
