File: KiCad 9 ESP32 demo project/User_Interface.kicad_sch (KiCad schematic)
At the start: 0 parts

Commit message: Schematic Done
Parts:
- added C21: 0.1U, Resistor_SMD:R_0805_2012Metric, symbol Device:C
- added C22: 1u, Resistor_SMD:R_0805_2012Metric, symbol Device:C
- added J4: Conn_01x04_Pin, Connector_PinHeader_2.54mm:PinHeader_1x04_P2.54mm_Vertical, symbol Connector:Conn_01x04_Pin
- added J5: Conn_01x05_Pin, Connector_PinHeader_2.54mm:PinHeader_1x05_P2.54mm_Vertical, symbol Connector:Conn_01x05_Pin
- added Q2, Q3: BC817, Resistor_SMD:R_0805_2012Metric, symbol Transistor_BJT:BC817
- added R32, R33, R34: 10K, Resistor_SMD:R_0805_2012Metric, symbol Device:R
- added S1: RESET, USLPT2819DT2TR:SW_USLPT2819DT2TR, symbol USLPT2819DT2TR:USLPT2819DT2TR
- added S2: BOOT, USLPT2819DT2TR:SW_USLPT2819DT2TR, symbol USLPT2819DT2TR:USLPT2819DT2TR
Connections:
- new net: Q3.1 (B), R34.2
- new net: Q2.1 (B), R33.2
- new net +3.3V: J4.1 (Pin_1), J5.1 (Pin_1), R32.2
- new net BOOT: C21.1, Q3.2 (E), S2.3, S2.4
- new net DTR: Q3.3 (C), R33.1
- new net EN: C22.1, Q2.3 (C), R32.1, S1.3, S1.4
- new net GND: C21.2, C22.2, J4.4 (Pin_4), J5.5 (Pin_5), S1.1, S1.2, S2.1, S2.2
- new net GPIO18: J5.3 (Pin_3)
- new net GPIO19: J5.4 (Pin_4)
- new net GPIO8: J5.2 (Pin_2)
- new net RTS: Q2.2 (E), R34.1
- new net SCL: J4.3 (Pin_3)
- new net SDA: J4.2 (Pin_2)
Other:
- note added: "Breakout for remaining pins"
- note added: "OLED Display connector(I2C)"
- note added: "RESET and BOOT Buttons"

Commit message: stated layout
Parts:
- C21, C22: footprint Resistor_SMD:R_0805_2012Metric -> Capacitor_SMD:C_0805_2012Metric
- Q2, Q3: footprint Resistor_SMD:R_0805_2012Metric -> BC817:SOT95P230X110-3N
Other:
- moved on the sheet: J5
Changed lines of the file:
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@@
 	(wire
 		(pts
-			(xy 34.29 105.41) (xy 40.64 105.41)
+			(xy 34.29 104.14) (xy 40.64 104.14)
 		)
 		(stroke
@@
 	(wire
 		(pts
-			(xy 34.29 110.49) (xy 40.64 110.49)
+			(xy 34.29 109.22) (xy 40.64 109.22)
 		)
 		(stroke
@@
 	(wire
 		(pts
-			(xy 34.29 97.79) (xy 34.29 102.87)
+			(xy 34.29 96.52) (xy 34.29 101.6)
 		)
 		(stroke
@@
 	(wire
 		(pts
-			(xy 34.29 102.87) (xy 40.64 102.87)
+			(xy 34.29 101.6) (xy 40.64 101.6)
 		)
 		(stroke
@@
 	(wire
 		(pts
-			(xy 34.29 113.03) (xy 34.29 118.11)
+			(xy 34.29 111.76) (xy 34.29 116.84)
 		)
 		(stroke
@@
 	(wire
 		(pts
-			(xy 40.64 113.03) (xy 34.29 113.03)
+			(xy 40.64 111.76) (xy 34.29 111.76)
 		)
 		(stroke
@@
 	(wire
 		(pts
-			(xy 34.29 107.95) (xy 40.64 107.95)
+			(xy 34.29 106.68) (xy 40.64 106.68)
 		)
 		(stroke
@@
 	)
 	(rectangle
-		(start 24.13 90.17)
-		(end 63.5 127)
+		(start 24.13 88.9)
+		(end 63.5 125.73)
 		(stroke
 			(width 0)
@@
 	(text "Breakout for remaining pins\n"
 		(exclude_from_sim no)
-		(at 38.354 87.884 0)
+		(at 38.354 86.614 0)
 		(effects
 			(font
@@
 	(hierarchical_label "GPIO19"
 		(shape bidirectional)
-		(at 34.29 110.49 180)
+		(at 34.29 109.22 180)
 		(effects
 			(font
@@
 	(hierarchical_label "GPIO8"
 		(shape bidirectional)
-		(at 34.29 105.41 180)
+		(at 34.29 104.14 180)
 		(effects
 			(font
@@
 	(hierarchical_label "GPIO18"
 		(shape bidirectional)
-		(at 34.29 107.95 180)
+		(at 34.29 106.68 180)
 		(effects
 			(font
@@
 			)
 		)
-		(property "Footprint" "Resistor_SMD:R_0805_2012Metric"
+		(property "Footprint" "Capacitor_SMD:C_0805_2012Metric"
 			(at 88.5952 72.39 0)
 			(effects
@@
 			)
 		)
-		(property "Footprint" "Resistor_SMD:R_0805_2012Metric"
+		(property "Footprint" "BC817:SOT95P230X110-3N"
 			(at 124.46 123.825 0)
 			(effects
@@
 	(symbol
 		(lib_id "power:+3.3V")
-		(at 34.29 97.79 0)
+		(at 34.29 96.52 0)
 		(unit 1)
 		(exclude_from_sim no)
@@
 		(fields_autoplaced yes)
 		(property "Reference" "#PWR49"
-			(at 34.29 101.6 0)
+			(at 34.29 100.33 0)
 			(effects
 				(font
@@
 		)
 		(property "Value" "+3.3V"
-			(at 34.29 92.71 0)
+			(at 34.29 91.44 0)
 			(effects
 				(font
@@
 		)
 		(property "Footprint" ""
-			(at 34.29 97.79 0)
+			(at 34.29 96.52 0)
 			(effects
 				(font
@@
 		)
 		(property "Datasheet" ""
-			(at 34.29 97.79 0)
+			(at 34.29 96.52 0)
 			(effects
 				(font
@@
 		)
 		(property "Description" "Power symbol creates a global label with name \"+3.3V\""
-			(at 34.29 97.79 0)
+			(at 34.29 96.52 0)
 			(effects
 				(font
@@
 	(symbol
 		(lib_id "Connector:Conn_01x05_Pin")
-		(at 45.72 107.95 0)
+		(at 45.72 106.68 0)
 		(mirror y)
 		(unit 1)
@@
 		(dnp no)
 		(property "Reference" "J5"
-			(at 46.99 109.2201 0)
+			(at 46.99 107.9501 0)
 			(effects
 				(font
@@
 		)
 		(property "Value" "Conn_01x05_Pin"
-			(at 46.99 106.6801 0)
+			(at 46.99 105.4101 0)
 			(effects
 				(font
@@
 		)
 		(property "Footprint" "Connector_PinHeader_2.54mm:PinHeader_1x05_P2.54mm_Vertical"
-			(at 45.72 107.95 0)
+			(at 45.72 106.68 0)
 			(effects
 				(font
@@
 		)
 		(property "Datasheet" "~"
-			(at 45.72 107.95 0)
+			(at 45.72 106.68 0)
 			(effects
 				(font
@@
 		)
 		(property "Description" "Generic connector, single row, 01x05, script generated"
-			(at 45.72 107.95 0)
+			(at 45.72 106.68 0)
 			(effects
 				(font
@@
 			)
 		)
-		(property "Footprint" "Resistor_SMD:R_0805_2012Metric"
+		(property "Footprint" "BC817:SOT95P230X110-3N"
 			(at 124.46 106.045 0)
 			(effects
@@
 	(symbol
 		(lib_id "power:GND")
-		(at 34.29 118.11 0)
+		(at 34.29 116.84 0)
 		(unit 1)
 		(exclude_from_sim no)
@@
 		(fields_autoplaced yes)
 		(property "Reference" "#PWR50"
-			(at 34.29 124.46 0)
+			(at 34.29 123.19 0)
 			(effects
 				(font
@@
 		)
 		(property "Value" "GND"
-			(at 34.29 123.19 0)
+			(at 34.29 121.92 0)
 			(effects
 				(font
@@
 		)
 		(property "Footprint" ""
-			(at 34.29 118.11 0)
+			(at 34.29 116.84 0)
 			(effects
 				(font
@@
 		)
 		(property "Datasheet" ""
-			(at 34.29 118.11 0)
+			(at 34.29 116.84 0)
 			(effects
 				(font
@@
 		)
 		(property "Description" "Power symbol creates a global label with name \"GND\" , ground"
-			(at 34.29 118.11 0)
+			(at 34.29 116.84 0)
 			(effects
 				(font
@@
 			)
 		)
-		(property "Footprint" "Resistor_SMD:R_0805_2012Metric"
+		(property "Footprint" "Capacitor_SMD:C_0805_2012Metric"
 			(at 135.5852 73.66 0)
 			(effects
