File: KiCad 9 ESP32 demo project/KiCad 9 ESP32 demo project.kicad_pcb (KiCad board)
At the start: 4 copper layers, 130.6 x 57.6 mm, 85 parts, among them J1 SS-52400-002, J2 B2B-PH-SM4-TB, J3 GSD090012SEU, J4 Conn_01x04_Pin, J5 Conn_01x05_Pin, Q1 TEMT6000X01, Q2 BC817, Q3 BC817, U1 BME280, U2 MAX4466EXK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

Commit message: power layout done
Parts:
- added REF**: MountingHole_2.5mm, MountingHole:MountingHole_2.5mm, F.Cu at (187.5, 51.5)
- added REF**: MountingHole_2.5mm, MountingHole:MountingHole_2.5mm, F.Cu at (220.0, 49.5)
- added REF**: MountingHole_2.5mm, MountingHole:MountingHole_2.5mm, F.Cu at (187.0, 71.0)
- F1: footprint Connector_PinHeader_2.54mm:PinHeader_1x04_P2.54mm_Vertical -> KiCad:FUSC3226X100N
- moved J4 78.5 mm to (211.6, 40.0), turned to -90 degrees
- moved J5 70.6 mm to (199.0, 40.0), turned to -90 degrees
- moved C3 63.4 mm to (200.8, 69.5), turned to 180 degrees
- moved VR1 56.3 mm to (200.8, 63.5), turned to 90 degrees
- moved C4 56.1 mm to (195.2, 64.0), turned to -90 degrees
- moved C2 55.6 mm to (200.8, 72.0), turned to 180 degrees
- moved TP2 54.9 mm to (230.5, 70.9)
- moved TP4 51.0 mm to (275.5, 58.5)
- moved R2 50.4 mm to (204.0, 81.4), turned to 90 degrees
- moved R1 49.4 mm to (201.5, 81.4), turned to 90 degrees
- moved TP1 48.7 mm to (242.7, 61.0)
- moved C1 48.6 mm to (220.2, 78.3), turned to 90 degrees
- moved C11 45.9 mm to (227.4, 70.5)
- moved C20 45.7 mm to (214.5, 50.5), turned to 90 degrees
- moved C5 45.2 mm to (192.8, 64.0), turned to -90 degrees
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Routing:
- net GND: track 0.00 -> 141.7 mm, vias 0 -> 45
- net +3.3V: track 0.00 -> 77.8 mm, vias 0 -> 27
- net /ESP32-C3_02/MOSI_DI: track 0.00 -> 65.2 mm
- net /ESP32-C3_02/MISO_DO: track 0.00 -> 64.5 mm
- net /ESP32-C3_02/SCL: track 0.00 -> 63.7 mm, vias 0 -> 2
- net /ESP32-C3_02/SDA: track 0.00 -> 63.5 mm, vias 0 -> 2
- net /ESP32-C3_02/CS: track 0.00 -> 38.2 mm, vias 0 -> 2
- net /ESP32-C3_02/SCLK: track 0.00 -> 30.6 mm
- net /ESP32-C3_02/CS_SD: track 0.00 -> 30.2 mm, vias 0 -> 2
- net +5V: track 0.00 -> 29.9 mm
- net /+5V_USB: track 0.00 -> 15.0 mm, vias 0 -> 10
- net /USB_DP: track 0.00 -> 10.5 mm, vias 0 -> 1
- net /USB_DN: track 0.00 -> 10.5 mm, vias 0 -> 1
- net /VBUS: track 0.00 -> 10.3 mm, vias 0 -> 6
- net /VBAT: track 0.00 -> 8.81 mm
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- added copper zone on F.Cu, net +3.3V
- added copper zone on In1.Cu, net +3.3V
- added copper zone on F.Cu, net +5V
- added copper zone on F.Cu, net /+5V_USB
- added copper zone on In1.Cu, net /+5V_USB
- added copper zone on F.Cu, net /VBAT
- added copper zone on F.Cu, net /VBUS
- added copper zone on In1.Cu, net /VBUS
- added copper zone on F.Cu, net GND
- added copper zone on In2.Cu, net GND
Other:
- board size 130.6 x 57.6 mm -> 80.5 x 57.6 mm
- board text added: "0.2000 mm / 0.0000 mm"
- board text added: "0.3000 mm"
- board text added: "1.6000 mm"
- board text added: "4"
- board text added: "80.4960 mm x 57.6178 mm"
- board text added: "BOARD CHARACTERISTICS"
- board text added: "Board Thickness:"
- board text added: "Board overall dimensions:"
- board text added: "Castellated pads:"
- board text added: "Copper Finish:"
- board text added: "Copper Layer Count:"
- board text added: "Edge card connectors:"
- board text added: "Impedance Control:"
- board text added: "Min hole diameter:"
- board text added: "Min track/spacing:"
- board text added: "No"
- board text added: "None"
- board text added: "Plated Board Edge:"

Commit message: power layout done
Parts:
- moved TP4 18.2 mm to (262.6, 45.6)
Routing:
- net /ESP32-C3_02/CS_SD: track 30.2 -> 32.0 mm
Changed lines of the file:
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@@
 	(footprint "TestPoint:TestPoint_Pad_D1.0mm"
 		(layer "F.Cu")
-		(at 275.5 58.5)
+		(at 262.65 45.65)
 		(descr "SMD pad as test Point, diameter 1.0mm")
 		(tags "test point SMD pad")
@@
 	)
 	(segment
-		(start 261.45 44.5)
-		(end 262.15 45.2)
+		(start 257.9875 64.9125)
+		(end 255.5 64.9125)
 		(width 0.2)
 		(layer "F.Cu")
@@
 	)
 	(segment
-		(start 259.29 44.5)
+		(start 263.5 46.55)
 		(end 261.45 44.5)
 		(width 0.2)
@@
 	)
 	(segment
-		(start 262.15 45.2)
-		(end 262.2 45.2)
+		(start 261.45 44.5)
+		(end 259.29 44.5)
 		(width 0.2)
 		(layer "F.Cu")
@@
 	)
 	(segment
-		(start 257.9875 64.9125)
-		(end 255.5 64.9125)
+		(start 259.15 63.75)
+		(end 257.9875 64.9125)
 		(width 0.2)
 		(layer "F.Cu")
@@
 	)
 	(segment
-		(start 259.15 63.75)
-		(end 257.9875 64.9125)
+		(start 263.5 46.55)
+		(end 262.2 45.25)
+		(width 0.2)
+		(layer "F.Cu")
+		(net 28)
+	)
+	(segment
+		(start 262.2 45.25)
+		(end 262.2 45.2)
 		(width 0.2)
 		(layer "F.Cu")
@@
 	)
 	(via
-		(at 262.15 45.2)
+		(at 263.5 46.55)
 		(size 0.5)
 		(drill 0.3)
@@
 	)
 	(segment
-		(start 262.15 45.2)
-		(end 263.5 46.55)
-		(width 0.2)
-		(layer "B.Cu")
-		(net 28)
-	)
-	(segment
 		(start 263.5 62.75)
-		(end 262.6 63.65)
+		(end 262.5 63.75)
 		(width 0.2)
 		(layer "B.Cu")
@@
 		(width 0.2)
 		(layer "B.Cu")
-		(net 28)
-	)
-	(segment
-		(start 262.6 63.65)
-		(end 262.5 63.75)
-		(width 0.2)
-		(layer "B.Cu")
